Commit message: working dynamic model

File: src/arm/urdf/arm_core.urdf.xacro (robot description, xacro)
@@ -49,15 +49,15 @@
     <inertial>
       <origin
-        xyz="4.09291668656414E-06 0.00280757977321831 -0.0263769532908136"
-        rpy="0 0 0" />
-      <mass
-        value="0.913798575246718" />
-      <inertia
-        ixx="0.000738791751701404"
-        ixy="-5.75329601726248E-09"
-        ixz="2.80419912699289E-08"
-        iyy="0.0011562373940488"
-        iyz="8.50224940441207E-08"
-        izz="0.000841350922681244" />
+        xyz="0.000006 0.001114 -0.019768"
+        rpy="0 0 0" />
+      <mass
+        value="1.889" />
+      <inertia
+        ixx="0.003485053"
+        ixy="-0.000000287"
+        ixz="0.000000106"
+        iyy="0.004329710"
+        iyz="0.000035555"
+        izz="0.001983100"/>
     </inertial>
     <visual>
@@ -107,15 +107,15 @@
     <inertial>
       <origin
-        xyz="0.295660685573248 1.97339206087221E-09 0.0632129424708848"
-        rpy="0 0 0" />
-      <mass
-        value="0.380008611681788" />
-      <inertia
-        ixx="0.000175559418519974"
-        ixy="9.72369978687692E-11"
-        ixz="-4.801848839621E-06"
-        iyy="0.00300845122180772"
-        iyz="-1.30095166425468E-11"
-        izz="0.00305616555189797" />
+        xyz="0.404172 0.000000 0.048931"
+        rpy="0 0 0" />
+      <mass
+        value="0.818" />
+      <inertia
+        ixx="0.000825516"
+        ixy="-0.000000001"
+        ixz="-0.001442463"
+        iyy="0.063324330"
+        iyz="0.000000000"
+        izz="0.062951082"/>
     </inertial>
     <visual>
@@ -165,15 +165,15 @@
     <inertial>
       <origin
-        xyz="0.0263064294366529 0.146366952173937 -0.00805675482743204"
-        rpy="0 0 0" />
-      <mass
-        value="0.238605745340086" />
-      <inertia
-        ixx="0.00218726998909511"
-        ixy="-8.98624821265651E-09"
-        ixz="1.95850088437551E-06"
-        iyy="0.000112084445050758"
-        iyz="-7.72526188677785E-11"
-        izz="0.00227353669762659" />
+        xyz="0.037731 0.362260 -0.001888"
+        rpy="0 0 0" />
+      <mass
+        value="0.537" />
+      <inertia
+        ixx="0.022532593"
+        ixy="0.001272152"
+        ixz="0.000062364"
+        iyy="0.000351160"
+        iyz="0.000594673"
+        izz="0.022677241"/>
     </inertial>
     <visual>
@@ -223,15 +223,15 @@
     <inertial>
       <origin
-        xyz="-7.52958278054938E-05 -0.000161441625529002 -0.00285726554010637"
-        rpy="0 0 0" />
-      <mass
-        value="0.0708022799545759" />
-      <inertia
-        ixx="1.41353753540356E-05"
-        ixy="7.97726994775567E-09"
-        ixz="-1.56574444311003E-10"
-        iyy="1.96983268044385E-05"
-        iyz="-4.01928980634711E-09"
-        izz="1.44656767445609E-05" />
+        xyz="-0.000088 -0.002372 -0.001219"
+        rpy="0 0 0" />
+      <mass
+        value="0.166" />
+      <inertia
+        ixx="0.000047749"
+        ixy="-0.000000202"
+        ixz="-0.000000016"
+        iyy="0.000049707"
+        iyz="-0.000001853"
+        izz="0.000043500"/>
     </inertial>
     <visual>
@@ -281,15 +281,15 @@
     <inertial>
       <origin
-        xyz="-4.73726066568814E-08 -0.0259717682743559 0.0246559410060783"
-        rpy="0 0 0" />
-      <mass
-        value="0.0651571805551386" />
-      <inertia
-        ixx="1.23629405434362E-05"
-        ixy="-3.13170044403038E-10"
-        ixz="-2.81505338860848E-11"
-        iyy="1.49174929347889E-05"
-        iyz="-1.06785390094496E-09"
-        izz="8.59424820964246E-06" />
+        xyz="-0.000001 -0.020304 0.038224"
+        rpy="0 0 0" />
+      <mass
+        value="0.134" />
+      <inertia
+        ixx="0.000096108"
+        ixy="0.000000000"
+        ixz="-0.000000001"
+        iyy="0.000074144"
+        iyz="0.000019325"
+        izz="0.000038048"/>
     </inertial>
     <visual>
@@ -339,15 +339,15 @@
     <inertial>
       <origin
-        xyz="5.55111512312578E-17 0 -0.00485640090169481"
-        rpy="0 0 0" />
-      <mass
-        value="0.0245056804431765" />
-      <inertia
-        ixx="3.15824905363328E-06"
-        ixy="2.02182651870993E-21"
-        ixz="-3.17953134358005E-22"
-        iyy="3.15824905363328E-06"
-        iyz="-5.13990365328799E-22"
-        izz="5.68068244515307E-06" />
+        xyz="0.000000 0.000000 -0.004856"
+        rpy="0 0 0" />
+      <mass
+        value="0.025" />
+      <inertia
+        ixx="0.000003158"
+        ixy="0.000000000"
+        ixz="0.000000000"
+        iyy="0.000003158"
+        iyz="0.000000000"
+        izz="0.000005681"/>
     </inertial>
     <visual>

File: src/arm/urdf/grippers/my_gripper_1.urdf.xacro (robot description, xacro)
@@ -14,15 +14,15 @@
     <inertial>
       <origin
-        xyz="-0.00247570175891211 0.00192421013672114 0.0748513008412715"
+        xyz="-0.002632 0.001808 0.074747"
         rpy="0 0 0" />
       <mass
         value="0.0983878201165868" />
       <inertia
-        ixx="0.000105485313306803"
-        ixy="-2.1042248306272E-08"
-        ixz="-9.20933039542333E-07"
-        iyy="0.000114758918473628"
-        iyz="1.1047801985657E-08"
-        izz="1.15747438919022E-05" />
+        ixx="0.000206703"
+        ixy="-0.000000132"
+        ixz="-0.000001890"
+        iyy="0.000213882"
+        iyz="0.000008203"
+        izz="0.000014312"/>
     </inertial>
     <visual>
@@ -54,15 +54,15 @@
     <inertial>
       <origin
-        xyz="-0.0168280191021532 0.0281845595187908 0.00070564854294175"
+        xyz="-0.044520 0.010236 -0.002794"
         rpy="0 0 0" />
       <mass
         value="0.054318578390507" />
       <inertia
-        ixx="2.00880186030608E-05"
-        ixy="1.65175563360546E-05"
-        ixz="-4.99481154962564E-08"
-        iyy="2.16573207842977E-05"
-        iyz="8.1654898204742E-08"
-        izz="4.12786244534564E-05" />
+        ixx="0.000023200"
+        ixy="-0.000019023"
+        ixz="0.000002080"
+        iyy="0.000026548"
+        iyz="-0.000001423"
+        izz="0.000046725"/>
     </inertial>
     <visual>

File: src/arm_moveit_config/config/arm.ros2_control.xacro (robot description, xacro)
@@ -23,4 +23,10 @@
     <xacro:arg name="stm32_feedback_wait_timeout_sec" default="2.0"/>
     <xacro:arg name="enable_stm32_zero_trigger" default="false"/>
+    <xacro:arg name="stm32_trace_enabled" default="false"/>
+    <xacro:arg name="stm32_trace_directory" default="/tmp/arm_stm32_traces"/>
+    <xacro:arg name="stm32_trace_run_label" default=""/>
+    <xacro:arg name="stm32_trace_file" default=""/>
+    <xacro:arg name="stm32_trace_append" default="false"/>
+    <xacro:arg name="stm32_trace_decimation" default="1"/>
     <xacro:arg name="enable_dynamics_feedforward" default="false"/>
     <xacro:arg name="dynamics_mode" default="gravity"/>
@@ -71,4 +77,10 @@
         stm32_feedback_wait_timeout_sec:='2.0'
         enable_stm32_zero_trigger:='false'
+        stm32_trace_enabled:='false'
+        stm32_trace_directory:='/tmp/arm_stm32_traces'
+        stm32_trace_run_label:=''
+        stm32_trace_file:=''
+        stm32_trace_append:='false'
+        stm32_trace_decimation:='1'
         enable_dynamics_feedforward:='false'
         dynamics_mode:='gravity'
@@ -111,4 +123,10 @@
                     <param name="stm32_feedback_wait_timeout_sec">${stm32_feedback_wait_timeout_sec}</param>
                     <param name="enable_stm32_zero_trigger">${enable_stm32_zero_trigger}</param>
+                    <param name="stm32_trace_enabled">${stm32_trace_enabled}</param>
+                    <param name="stm32_trace_directory">${stm32_trace_directory}</param>
+                    <param name="stm32_trace_run_label">${stm32_trace_run_label}</param>
+                    <param name="stm32_trace_file">${stm32_trace_file}</param>
+                    <param name="stm32_trace_append">${stm32_trace_append}</param>
+                    <param name="stm32_trace_decimation">${stm32_trace_decimation}</param>
                     <param name="enable_dynamics_feedforward">${enable_dynamics_feedforward}</param>
                     <param name="dynamics_mode">${dynamics_mode}</param>
@@ -128,5 +146,5 @@
             <xacro:position_joint_interfaces joint_name="joint_3" initial_value="${initial_positions['joint_3']}" min_limit="-3.14" max_limit="0.0"/>
             <xacro:position_joint_interfaces joint_name="joint_4" initial_value="${initial_positions['joint_4']}" min_limit="-3.14" max_limit="3.14"/>
-            <xacro:position_joint_interfaces joint_name="joint_5" initial_value="${initial_positions['joint_5']}" min_limit="0.0" max_limit="3.14"/>
+            <xacro:position_joint_interfaces joint_name="joint_5" initial_value="${initial_positions['joint_5']}" min_limit="0" max_limit="3.14"/>
             <xacro:position_joint_interfaces joint_name="joint_6" initial_value="${initial_positions['joint_6']}" min_limit="-3.14" max_limit="3.14"/>
             <xacro:position_joint_interfaces joint_name="tool_joint" initial_value="${initial_positions['tool_joint']}" min_limit="${aux_joint_min}" max_limit="${aux_joint_max}"/>

File: src/arm_moveit_config/config/arm.urdf.xacro (robot description, xacro)
@@ -24,4 +24,10 @@
     <xacro:arg name="stm32_feedback_wait_timeout_sec" default="2.0" />
     <xacro:arg name="enable_stm32_zero_trigger" default="false" />
+    <xacro:arg name="stm32_trace_enabled" default="false" />
+    <xacro:arg name="stm32_trace_directory" default="/tmp/arm_stm32_traces" />
+    <xacro:arg name="stm32_trace_run_label" default="" />
+    <xacro:arg name="stm32_trace_file" default="" />
+    <xacro:arg name="stm32_trace_append" default="false" />
+    <xacro:arg name="stm32_trace_decimation" default="1" />
     <xacro:arg name="enable_dynamics_feedforward" default="false" />
     <xacro:arg name="dynamics_mode" default="gravity" />
@@ -91,4 +97,10 @@
       stm32_feedback_wait_timeout_sec="$(arg stm32_feedback_wait_timeout_sec)"
       enable_stm32_zero_trigger="$(arg enable_stm32_zero_trigger)"
+      stm32_trace_enabled="$(arg stm32_trace_enabled)"
+      stm32_trace_directory="$(arg stm32_trace_directory)"
+      stm32_trace_run_label="$(arg stm32_trace_run_label)"
+      stm32_trace_file="$(arg stm32_trace_file)"
+      stm32_trace_append="$(arg stm32_trace_append)"
+      stm32_trace_decimation="$(arg stm32_trace_decimation)"
       enable_dynamics_feedforward="$(arg enable_dynamics_feedforward)"
       dynamics_mode="$(arg dynamics_mode)"
