Commit message: 1

File: src/arm/urdf/arm.urdf (robot description, URDF)
Before this commit: robot arm, 10 links, 9 joints
Joints:
- joint joint2: limit lower=0.00 upper=3.14 effort=0 velocity=2.0 -> lower=0 upper=3.14 effort=0 velocity=2.0
- joint joint5: limit lower=-0.1 upper=3.14 effort=0 velocity=2.0 -> lower=0 upper=3.14 effort=0 velocity=2.0
- joint tool0_fixed: origin xyz=-0.02 0 0.15 rpy=0 -0.30 0 -> xyz=-0.02 0 0.15 rpy=0 -0.3 0

File: src/arm_moveit_config/config/arm.ros2_control.xacro (robot description, xacro)
@@ -60,7 +60,6 @@
             <joint name="joint5">
                 <command_interface name="position"/>
-                  <param name="min"> -0.1 </param>
+                  <param name="min"> 0 </param>
                   <param name="max"> 3.14</param>
-                  <param name="max"> 1.3</param>
                 <state_interface name="position">
                   <param name="initial_value">${initial_positions['joint5']}</param>

Commit message: latest

File: src/arm/urdf/arm.urdf (robot description, URDF)
Before this commit: robot arm, 10 links, 9 joints
Links:
- removed link link1
- removed link link2
- removed link link3
- removed link link4
- removed link link5
- removed link link6
- removed link link7
- added link link_1, mass 0.82985; collision mesh filename=package://arm/meshes/link_1.STL; visual mesh filename=package://arm/meshes/link_1.STL
- added link link_2, mass 0.78271; collision mesh filename=package://arm/meshes/link_2.STL; visual mesh filename=package://arm/meshes/link_2.STL
- added link link_3, mass 0.12605; collision mesh filename=package://arm/meshes/link_3.STL; visual mesh filename=package://arm/meshes/link_3.STL
- added link link_4, mass 0.067165; collision mesh filename=package://arm/meshes/link_4.STL; visual mesh filename=package://arm/meshes/link_4.STL
- added link link_5, mass 0.060361; collision mesh filename=package://arm/meshes/link_5.STL; visual mesh filename=package://arm/meshes/link_5.STL
- added link link_6, mass 0.12546; collision mesh filename=package://arm/meshes/link_6.STL; visual mesh filename=package://arm/meshes/link_6.STL
- added link tool_link, mass 0.054319; collision mesh filename=package://arm/meshes/tool_link.STL; visual mesh filename=package://arm/meshes/tool_link.STL
- link base_link: mass 0.13398639623737 -> 0.32006
- link tool0: geometry 
Joints:
- removed joint joint1
- removed joint joint2
- removed joint joint3
- removed joint joint4
- removed joint joint5
- removed joint joint6
- removed joint joint7
- added joint joint_1: type revolute, parent base_link, child link_1, origin xyz=0 0 0.105 rpy=0 0 0, axis 0 0 -1, limit lower=-3.14 upper=3.14 effort=0 velocity=2.0
- added joint joint_2: type revolute, parent link_1, child link_2, origin xyz=0.092 0 0 rpy=1.5708 0 1.5708, axis 0 0 1, limit lower=-3.14 upper=3.14 effort=0 velocity=2.0
- added joint joint_3: type revolute, parent link_2, child link_3, origin xyz=0.65 0 -0.036 rpy=-3.1416 0 1.5708, axis 0 0 1, limit lower=-3.14 upper=3.14 effort=0 velocity=2.0
- added joint joint_4: type revolute, parent link_3, child link_4, origin xyz=0.045 -0.566 0 rpy=-1.5708 0 3.1416, axis 0 0 1, limit lower=-3.14 upper=3.14 effort=0 velocity=2.0
- added joint joint_5: type revolute, parent link_4, child link_5, origin xyz=0 0 0 rpy=1.5708 0 -1.5708, axis 0 0 -1, limit lower=-3.14 upper=3.14 effort=0 velocity=2.0
- added joint joint_6: type revolute, parent link_5, child link_6, origin xyz=0 0 0 rpy=1.5708 0 1.5708, axis 0 0 1, limit lower=-3.14 upper=3.14 effort=0 velocity=2.0
- added joint tool_joint: type revolute, parent link_6, child tool_link, origin xyz=-0.02305 0.00055 0.138 rpy=-1.5708 0 -3.1416, axis 0 0 1, limit lower=-3.14 upper=3.14 effort=0 velocity=2.0
- joint tool0_fixed: origin xyz=-0.02 0 0.15 rpy=0 -0.3 0 -> xyz=0 0 0 rpy=0 0 0; parent link6 -> tool_link

File: src/arm_moveit_config/config/arm.ros2_control.xacro (robot description, xacro)
@@ -1,96 +1,91 @@
 <?xml version="1.0"?>
 <robot xmlns:xacro="http://www.ros.org/wiki/xacro">
-    <xacro:arg name="hw_plugin" default="my_arm_hardware/MyArmSystem"/>
-    <!-- <plugin>mock_components/GenericSystem</plugin> -->
-    <xacro:arg name="serial_port" default="/dev/ttyUSB0"/>
-    <xacro:arg name="baudrate" default="115200"/>
-    <xacro:macro name="arm_ros2_control" params="name initial_positions_file">
+    <xacro:arg name="use_fake_hardware" default="true"/>
+    <xacro:arg name="serial_port" default="/dev/ttyUSB4"/>
+    <xacro:arg name="reader_port" default="/dev/ttyUSB5"/>
+    <xacro:arg name="gripper_port" default="/dev/ttyUSB6"/>
+    <xacro:arg name="baudrate" default="230400"/>
+    <xacro:arg name="gripper_baudrate" default="115200"/>
+    <xacro:arg name="position_scale" default="1000"/>
+    <xacro:arg name="hw_slowdown" default="10"/>
+    <xacro:arg name="initial_read_timeout_sec" default="2.0"/>
+    <xacro:arg name="aux_joint_min" default="-3.14"/>
+    <xacro:arg name="aux_joint_max" default="3.14"/>
+    <xacro:arg name="enable_feedback_plot" default="false"/>
+    <xacro:arg name="feedback_plot_rate_hz" default="100"/>
+    <xacro:arg name="feedback_plot_min_rad" default="-1.0"/>
+    <xacro:arg name="feedback_plot_max_rad" default="1.0"/>
+    <xacro:arg name="feedback_plot_joint_filter" default="joint_1,joint_2,joint_3"/>
+    <xacro:arg name="feedback_plot_csv_enabled" default="false"/>
+    <xacro:arg name="feedback_plot_csv_file" default="/tmp/joint_monitor.csv"/>
+    <xacro:arg name="feedback_plot_csv_append" default="false"/>
+    <xacro:macro name="position_joint_interfaces" params="joint_name initial_value min_limit max_limit">
+        <joint name="${joint_name}">
+            <command_interface name="position"/>
+            <param name="min">${min_limit}</param>
+            <param name="max">${max_limit}</param>
+            <state_interface name="position">
+                <param name="initial_value">${initial_value}</param>
+            </state_interface>
+            <state_interface name="velocity"/>
+        </joint>
+    </xacro:macro>
+    <xacro:macro name="arm_ros2_control" params="
+        name
+        initial_positions_file
+        use_fake_hardware:=true
+        serial_port:='/dev/ttyUSB4'
+        reader_port:='/dev/ttyUSB5'
+        gripper_port:='/dev/ttyUSB6'
+        baudrate:='230400'
+        gripper_baudrate:='115200'
+        position_scale:='1000'
+        hw_slowdown:='10'
+        initial_read_timeout_sec:='2.0'
+        aux_joint_min:='-3.14'
+        aux_joint_max:='3.14'
+        enable_feedback_plot:='false'
+        feedback_plot_rate_hz:='100'
+        feedback_plot_min_rad:='-1.0'
+        feedback_plot_max_rad:='1.0'
+        feedback_plot_joint_filter:='joint_1,joint_2,joint_3'
+        feedback_plot_csv_enabled:='false'
+        feedback_plot_csv_file:='/tmp/joint_monitor.csv'
+        feedback_plot_csv_append:='false'">
         <xacro:property name="initial_positions" value="${xacro.load_yaml(initial_positions_file)['initial_positions']}"/>
-        <!-- <xacro:arg name="hw_plugin" default="mock_components/GenericSystem"/> -->
         <ros2_control name="${name}" type="system">
             <hardware>
-                <!-- By default, set up controllers for simulation. This won't work on real hardware -->
-                <!-- <plugin>mock_components/GenericSystem</plugin> -->
-                <plugin>my_arm_hardware/MyArmHardware</plugin>
-                <param name="serial_port">/dev/ttyUSB4</param>
-                <param name="reader_port">/dev/ttyUSB5</param>
-                <param name="gripper_port">/dev/ttyUSB6</param>
-                <param name="baudrate">230400</param>
-                <param name="gripper_baudrate">115200</param>
-                <param name="position_scale">1000</param>
-                <param name="hw_slowdown">10</param>
-                <param name="initial_read_timeout_sec">2.0</param>
-                <param name="enable_feedback_plot">true</param>
-                <param name="feedback_plot_rate_hz">100</param>
-                <param name="feedback_plot_min_rad">-1.</param>
-                <param name="feedback_plot_max_rad">1.</param>
-                <param name="feedback_plot_joint_filter">joint1,joint2,joint3</param>
-                <param name="feedback_plot_csv_enabled">true</param>
-                <param name="feedback_plot_csv_file">/tmp/joint_monitor.csv</param>
-                <param name="feedback_plot_csv_append">false</param>
+                <xacro:if value="${use_fake_hardware}">
+                    <plugin>mock_components/GenericSystem</plugin>
+                </xacro:if>
+                <xacro:unless value="${use_fake_hardware}">
+                    <plugin>my_arm_hardware/MyArmHardware</plugin>
+                    <param name="serial_port">${serial_port}</param>
+                    <param name="reader_port">${reader_port}</param>
+                    <param name="gripper_port">${gripper_port}</param>
+                    <param name="baudrate">${baudrate}</param>
+                    <param name="gripper_baudrate">${gripper_baudrate}</param>
+                    <param name="position_scale">${position_scale}</param>
+                    <param name="hw_slowdown">${hw_slowdown}</param>
+                    <param name="initial_read_timeout_sec">${initial_read_timeout_sec}</param>
+                    <param name="aux_joint_min">${aux_joint_min}</param>
+                    <param name="aux_joint_max">${aux_joint_max}</param>
+                    <param name="enable_feedback_plot">${enable_feedback_plot}</param>
+                    <param name="feedback_plot_rate_hz">${feedback_plot_rate_hz}</param>
+                    <param name="feedback_plot_min_rad">${feedback_plot_min_rad}</param>
+                    <param name="feedback_plot_max_rad">${feedback_plot_max_rad}</param>
+                    <param name="feedback_plot_joint_filter">${feedback_plot_joint_filter}</param>
+                    <param name="feedback_plot_csv_enabled">${feedback_plot_csv_enabled}</param>
+                    <param name="feedback_plot_csv_file">${feedback_plot_csv_file}</param>
+                    <param name="feedback_plot_csv_append">${feedback_plot_csv_append}</param>
+                </xacro:unless>
             </hardware>
-            <joint name="joint1">
-                <command_interface name="position"/>
-                  <param name="min"> -1.57</param>
-                  <param name="max"> 1.57</param>
-                <state_interface name="position">
-                  <param name="initial_value">${initial_positions['joint1']}</param>
-                </state_interface>
-                <state_interface name="velocity"/>
-            </joint>
-            <joint name="joint2">
-                <command_interface name="position"/>
-                  <param name="min"> 0.00</param>
-                  <param name="max"> 3.14</param>
-                <state_interface name="position">
-                  <param name="initial_value">${initial_positions['joint2']}</param>
-                </state_interface>
-                <state_interface name="velocity"/>
-            </joint>
-            <joint name="joint3">
-                <command_interface name="position"/>
-                  <param name="min"> -3.14 </param>
-                  <param name="max"> 0.00</param>
-                <state_interface name="position">
-                  <param name="initial_value">${initial_positions['joint3']}</param>
-                </state_interface>
-                <state_interface name="velocity"/>
-            </joint>
-            <joint name="joint4">
-                <command_interface name="position"/>
-                  <param name="min"> -3.14 </param>
-                  <param name="max"> 3.14</param>
-                <state_interface name="position">
-                  <param name="initial_value">${initial_positions['joint4']}</param>
-                </state_interface>
-                <state_interface name="velocity"/>
-            </joint>
-            <joint name="joint5">
-                <command_interface name="position"/>
-                  <param name="min"> 0 </param>
-                  <param name="max"> 3.14</param>
-                <state_interface name="position">
-                  <param name="initial_value">${initial_positions['joint5']}</param>
-                </state_interface>
-                <state_interface name="velocity"/>
-            </joint>
-            <joint name="joint6">
-                <command_interface name="position"/>
-                  <param name="min"> -3.14 </param>
-                  <param name="max"> 3.14</param>
-                <state_interface name="position">
-                  <param name="initial_value">${initial_positions['joint6']}</param>
-                </state_interface>
-                <state_interface name="velocity"/>
-            </joint>
-            <joint name="joint7">
-                <command_interface name="position"/>
-                  <param name="min"> -0.69 </param>
-                  <param name="max"> 0.00</param>
-                <state_interface name="position">
-                  <param name="initial_value">${initial_positions['joint7']}</param>
-                </state_interface>
-                <state_interface name="velocity"/>
-            </joint>
+            <xacro:position_joint_interfaces joint_name="joint_1" initial_value="${initial_positions['joint_1']}" min_limit="-3.14" max_limit="3.14"/>
+            <xacro:position_joint_interfaces joint_name="joint_2" initial_value="${initial_positions['joint_2']}" min_limit="-3.14" max_limit="3.14"/>
+            <xacro:position_joint_interfaces joint_name="joint_3" initial_value="${initial_positions['joint_3']}" min_limit="-3.14" max_limit="3.14"/>
+            <xacro:position_joint_interfaces joint_name="joint_4" initial_value="${initial_positions['joint_4']}" min_limit="-3.14" max_limit="3.14"/>
+            <xacro:position_joint_interfaces joint_name="joint_5" initial_value="${initial_positions['joint_5']}" min_limit="-3.14" max_limit="3.14"/>
+            <xacro:position_joint_interfaces joint_name="joint_6" initial_value="${initial_positions['joint_6']}" min_limit="-3.14" max_limit="3.14"/>
+            <xacro:position_joint_interfaces joint_name="tool_joint" initial_value="${initial_positions['tool_joint']}" min_limit="${aux_joint_min}" max_limit="${aux_joint_max}"/>
         </ros2_control>
     </xacro:macro>

File: src/arm_moveit_config/config/arm.urdf.xacro (robot description, xacro)
@@ -2,4 +2,23 @@
 <robot xmlns:xacro="http://www.ros.org/wiki/xacro" name="arm">
     <xacro:arg name="initial_positions_file" default="initial_positions.yaml" />
+    <xacro:arg name="use_fake_hardware" default="true" />
+    <xacro:arg name="serial_port" default="/dev/ttyUSB4" />
+    <xacro:arg name="reader_port" default="/dev/ttyUSB5" />
+    <xacro:arg name="gripper_port" default="/dev/ttyUSB6" />
+    <xacro:arg name="baudrate" default="230400" />
+    <xacro:arg name="gripper_baudrate" default="115200" />
+    <xacro:arg name="position_scale" default="1000" />
+    <xacro:arg name="hw_slowdown" default="10" />
+    <xacro:arg name="initial_read_timeout_sec" default="2.0" />
+    <xacro:arg name="aux_joint_min" default="-3.14" />
+    <xacro:arg name="aux_joint_max" default="3.14" />
+    <xacro:arg name="enable_feedback_plot" default="false" />
+    <xacro:arg name="feedback_plot_rate_hz" default="100" />
+    <xacro:arg name="feedback_plot_min_rad" default="-1.0" />
+    <xacro:arg name="feedback_plot_max_rad" default="1.0" />
+    <xacro:arg name="feedback_plot_joint_filter" default="joint_1,joint_2,joint_3" />
+    <xacro:arg name="feedback_plot_csv_enabled" default="false" />
+    <xacro:arg name="feedback_plot_csv_file" default="/tmp/joint_monitor.csv" />
+    <xacro:arg name="feedback_plot_csv_append" default="false" />
     <!-- Import arm urdf file -->
     <xacro:include filename="$(find arm)/urdf/arm.urdf" />
@@ -13,5 +32,5 @@
       parent_link="uav_mount"
       xyz="0 0 0.05"
-      rpy="0 0 0"
+      rpy="0 0 1.57"
       size="0.4 0.64 0.01"
       color="0.9 0.1 0.1 0.2"
@@ -20,6 +39,6 @@
       name="limit_y_min"
       parent_link="uav_mount"
-      xyz="0 -0.32 -0.8"
-      rpy="-1.57 0 0"
+      xyz="0.32 0 -0.75"
+      rpy="1.57 0 1.57"
       size="0.4 1.6 0.01"
       color="0.9 0.1 0.1 0.2"
@@ -28,9 +47,30 @@
       name="limit_y_max"
       parent_link="uav_mount"
-      xyz="0 0.32 -0.8"
-      rpy="1.57 0 0"
+      xyz="-0.32 0 -0.75"
+      rpy="1.57 0 1.57"
       size="0.4 1.6 0.01"
       color="0.9 0.1 0.1 0.2"
       collision_only="false"/>
-    <xacro:arm_ros2_control name="FakeSystem" initial_positions_file="$(arg initial_positions_file)"/>
+    <xacro:arm_ros2_control
+      name="ArmSystem"
+      initial_positions_file="$(arg initial_positions_file)"
+      use_fake_hardware="$(arg use_fake_hardware)"
+      serial_port="$(arg serial_port)"
+      reader_port="$(arg reader_port)"
+      gripper_port="$(arg gripper_port)"
+      baudrate="$(arg baudrate)"
+      gripper_baudrate="$(arg gripper_baudrate)"
+      position_scale="$(arg position_scale)"
+      hw_slowdown="$(arg hw_slowdown)"
+      initial_read_timeout_sec="$(arg initial_read_timeout_sec)"
+      aux_joint_min="$(arg aux_joint_min)"
+      aux_joint_max="$(arg aux_joint_max)"
+      enable_feedback_plot="$(arg enable_feedback_plot)"
+      feedback_plot_rate_hz="$(arg feedback_plot_rate_hz)"
+      feedback_plot_min_rad="$(arg feedback_plot_min_rad)"
+      feedback_plot_max_rad="$(arg feedback_plot_max_rad)"
+      feedback_plot_joint_filter="$(arg feedback_plot_joint_filter)"
+      feedback_plot_csv_enabled="$(arg feedback_plot_csv_enabled)"
+      feedback_plot_csv_file="$(arg feedback_plot_csv_file)"
+      feedback_plot_csv_append="$(arg feedback_plot_csv_append)"/>
 </robot>

Commit message: 1

File: src/arm/urdf/arm.urdf (robot description, URDF)
Before this commit: robot arm, 10 links, 9 joints
Joints:
- joint joint_2: limit lower=-3.14 upper=3.14 effort=0 velocity=2.0 -> lower=0.0 upper=3.14 effort=0 velocity=2.0
- joint joint_3: limit lower=-3.14 upper=3.14 effort=0 velocity=2.0 -> lower=0.0 upper=3.14 effort=0 velocity=2.0
- joint joint_5: limit lower=-3.14 upper=3.14 effort=0 velocity=2.0 -> lower=-3.14 upper=0.0 effort=0 velocity=2.0
- joint tool0_fixed: origin xyz=0 0 0 rpy=0 0 0 -> xyz=0 0.01 0.2 rpy=0 0 0; parent tool_link -> link_6

File: src/arm_moveit_config/config/arm.ros2_control.xacro (robot description, xacro)
@@ -9,4 +9,5 @@
     <xacro:arg name="position_scale" default="1000"/>
     <xacro:arg name="arm_joint_signs" default="1,1,-1,1,1,1"/>
+    <xacro:arg name="arm_joint_offsets" default="0,0,0,0,0,0"/>
     <xacro:arg name="hw_slowdown" default="10"/>
     <xacro:arg name="initial_read_timeout_sec" default="2.0"/>
@@ -44,4 +45,5 @@
         position_scale:='1000'
         arm_joint_signs:='1,1,-1,1,1,1'
+        arm_joint_offsets:='0,0,0,0,0,0'
         hw_slowdown:='10'
         initial_read_timeout_sec:='2.0'
@@ -72,4 +74,5 @@
                     <param name="position_scale">${position_scale}</param>
                     <param name="arm_joint_signs">${arm_joint_signs}</param>
+                    <param name="arm_joint_offsets">${arm_joint_offsets}</param>
                     <param name="hw_slowdown">${hw_slowdown}</param>
                     <param name="initial_read_timeout_sec">${initial_read_timeout_sec}</param>
@@ -88,8 +91,8 @@
             </hardware>
             <xacro:position_joint_interfaces joint_name="joint_1" initial_value="${initial_positions['joint_1']}" min_limit="-3.14" max_limit="3.14"/>
-            <xacro:position_joint_interfaces joint_name="joint_2" initial_value="${initial_positions['joint_2']}" min_limit="-3.14" max_limit="3.14"/>
-            <xacro:position_joint_interfaces joint_name="joint_3" initial_value="${initial_positions['joint_3']}" min_limit="-3.14" max_limit="3.14"/>
+            <xacro:position_joint_interfaces joint_name="joint_2" initial_value="${initial_positions['joint_2']}" min_limit="0.0" max_limit="3.14"/>
+            <xacro:position_joint_interfaces joint_name="joint_3" initial_value="${initial_positions['joint_3']}" min_limit="0.0" max_limit="3.14"/>
             <xacro:position_joint_interfaces joint_name="joint_4" initial_value="${initial_positions['joint_4']}" min_limit="-3.14" max_limit="3.14"/>
-            <xacro:position_joint_interfaces joint_name="joint_5" initial_value="${initial_positions['joint_5']}" min_limit="-3.14" max_limit="3.14"/>
+            <xacro:position_joint_interfaces joint_name="joint_5" initial_value="${initial_positions['joint_5']}" min_limit="-3.14" max_limit="0.0"/>
             <xacro:position_joint_interfaces joint_name="joint_6" initial_value="${initial_positions['joint_6']}" min_limit="-3.14" max_limit="3.14"/>
             <xacro:position_joint_interfaces joint_name="tool_joint" initial_value="${initial_positions['tool_joint']}" min_limit="${aux_joint_min}" max_limit="${aux_joint_max}"/>

File: src/arm_moveit_config/config/arm.urdf.xacro (robot description, xacro)
@@ -10,4 +10,5 @@
     <xacro:arg name="position_scale" default="1000" />
     <xacro:arg name="arm_joint_signs" default="1,1,-1,1,1,1" />
+    <xacro:arg name="arm_joint_offsets" default="0,0,0,0,0,0" />
     <xacro:arg name="hw_slowdown" default="10" />
     <xacro:arg name="initial_read_timeout_sec" default="2.0" />
@@ -65,4 +66,5 @@
       position_scale="$(arg position_scale)"
       arm_joint_signs="$(arg arm_joint_signs)"
+      arm_joint_offsets="$(arg arm_joint_offsets)"
       hw_slowdown="$(arg hw_slowdown)"
       initial_read_timeout_sec="$(arg initial_read_timeout_sec)"
