Commit message: dynamic estimation online

File: src/arm/urdf/arm.urdf (robot description, URDF)
Before this commit: robot arm, 10 links, 9 joints
Joints:
- joint tool_joint: limit lower=-3.14 upper=3.14 effort=0 velocity=2.0 -> lower=-0.69 upper=0.0 effort=0 velocity=2.0

File: src/arm_moveit_config/config/arm.ros2_control.xacro (robot description, xacro)
@@ -13,14 +13,18 @@
     <xacro:arg name="initial_read_timeout_sec" default="2.0"/>
     <xacro:arg name="first_power_on" default="true"/>
-    <xacro:arg name="aux_joint_min" default="-3.14"/>
-    <xacro:arg name="aux_joint_max" default="3.14"/>
-    <xacro:arg name="enable_feedback_plot" default="false"/>
-    <xacro:arg name="feedback_plot_rate_hz" default="100"/>
-    <xacro:arg name="feedback_plot_min_rad" default="-1.0"/>
-    <xacro:arg name="feedback_plot_max_rad" default="1.0"/>
-    <xacro:arg name="feedback_plot_joint_filter" default="joint_1,joint_2,joint_3"/>
-    <xacro:arg name="feedback_plot_csv_enabled" default="false"/>
-    <xacro:arg name="feedback_plot_csv_file" default="/tmp/joint_monitor.csv"/>
-    <xacro:arg name="feedback_plot_csv_append" default="false"/>
+    <xacro:arg name="aux_joint_min" default="-0.69"/>
+    <xacro:arg name="aux_joint_max" default="0.0"/>
+    <xacro:arg name="arm_command_frame_format" default="legacy_position"/>
+    <xacro:arg name="enable_dynamics_feedforward" default="false"/>
+    <xacro:arg name="dynamics_mode" default="gravity"/>
+    <xacro:arg name="dynamics_urdf_path" default=""/>
+    <xacro:arg name="dynamics_feedforward_source" default="topic"/>
+    <xacro:arg name="dynamics_feedforward_topic" default="/arm_dynamics/torques_nm"/>
+    <xacro:arg name="dynamics_topic_timeout_sec" default="0.25"/>
+    <xacro:arg name="dynamics_use_commanded_position" default="false"/>
+    <xacro:arg name="dynamics_torque_scale" default="1.0"/>
+    <xacro:arg name="dynamics_torque_limits_nm" default="0.5,0.5,0.3,0.2,0.15,0.1"/>
+    <xacro:arg name="dynamics_torque_joint_signs" default=""/>
+    <xacro:arg name="dynamics_torque_low_pass_alpha" default="0.2"/>
     <xacro:macro name="position_joint_interfaces" params="joint_name initial_value min_limit max_limit">
         <joint name="${joint_name}">
@@ -49,14 +53,18 @@
         initial_read_timeout_sec:='2.0'
         first_power_on:='true'
-        aux_joint_min:='-3.14'
-        aux_joint_max:='3.14'
-        enable_feedback_plot:='false'
-        feedback_plot_rate_hz:='100'
-        feedback_plot_min_rad:='-1.0'
-        feedback_plot_max_rad:='1.0'
-        feedback_plot_joint_filter:='joint_1,joint_2,joint_3'
-        feedback_plot_csv_enabled:='false'
-        feedback_plot_csv_file:='/tmp/joint_monitor.csv'
-        feedback_plot_csv_append:='false'">
+        aux_joint_min:='-0.69'
+        aux_joint_max:='0.0'
+        arm_command_frame_format:='legacy_position'
+        enable_dynamics_feedforward:='false'
+        dynamics_mode:='gravity'
+        dynamics_urdf_path:=''
+        dynamics_feedforward_source:='topic'
+        dynamics_feedforward_topic:='/arm_dynamics/torques_nm'
+        dynamics_topic_timeout_sec:='0.25'
+        dynamics_use_commanded_position:='false'
+        dynamics_torque_scale:='1.0'
+        dynamics_torque_limits_nm:='0.5,0.5,0.3,0.2,0.15,0.1'
+        dynamics_torque_joint_signs:=''
+        dynamics_torque_low_pass_alpha:='0.2'">
         <xacro:property name="initial_positions" value="${xacro.load_yaml(initial_positions_file)['initial_positions']}"/>
         <ros2_control name="${name}" type="system">
@@ -80,12 +88,16 @@
                     <param name="aux_joint_min">${aux_joint_min}</param>
                     <param name="aux_joint_max">${aux_joint_max}</param>
-                    <param name="enable_feedback_plot">${enable_feedback_plot}</param>
-                    <param name="feedback_plot_rate_hz">${feedback_plot_rate_hz}</param>
-                    <param name="feedback_plot_min_rad">${feedback_plot_min_rad}</param>
-                    <param name="feedback_plot_max_rad">${feedback_plot_max_rad}</param>
-                    <param name="feedback_plot_joint_filter">${feedback_plot_joint_filter}</param>
-                    <param name="feedback_plot_csv_enabled">${feedback_plot_csv_enabled}</param>
-                    <param name="feedback_plot_csv_file">${feedback_plot_csv_file}</param>
-                    <param name="feedback_plot_csv_append">${feedback_plot_csv_append}</param>
+                    <param name="arm_command_frame_format">${arm_command_frame_format}</param>
+                    <param name="enable_dynamics_feedforward">${enable_dynamics_feedforward}</param>
+                    <param name="dynamics_mode">${dynamics_mode}</param>
+                    <param name="dynamics_urdf_path">${dynamics_urdf_path}</param>
+                    <param name="dynamics_feedforward_source">${dynamics_feedforward_source}</param>
+                    <param name="dynamics_feedforward_topic">${dynamics_feedforward_topic}</param>
+                    <param name="dynamics_topic_timeout_sec">${dynamics_topic_timeout_sec}</param>
+                    <param name="dynamics_use_commanded_position">${dynamics_use_commanded_position}</param>
+                    <param name="dynamics_torque_scale">${dynamics_torque_scale}</param>
+                    <param name="dynamics_torque_limits_nm">${dynamics_torque_limits_nm}</param>
+                    <param name="dynamics_torque_joint_signs">${dynamics_torque_joint_signs}</param>
+                    <param name="dynamics_torque_low_pass_alpha">${dynamics_torque_low_pass_alpha}</param>
                 </xacro:unless>
             </hardware>

File: src/arm_moveit_config/config/arm.urdf.xacro (robot description, xacro)
@@ -14,14 +14,18 @@
     <xacro:arg name="initial_read_timeout_sec" default="2.0" />
     <xacro:arg name="first_power_on" default="true" />
-    <xacro:arg name="aux_joint_min" default="-3.14" />
-    <xacro:arg name="aux_joint_max" default="3.14" />
-    <xacro:arg name="enable_feedback_plot" default="false" />
-    <xacro:arg name="feedback_plot_rate_hz" default="100" />
-    <xacro:arg name="feedback_plot_min_rad" default="-1.0" />
-    <xacro:arg name="feedback_plot_max_rad" default="1.0" />
-    <xacro:arg name="feedback_plot_joint_filter" default="joint_1,joint_2,joint_3" />
-    <xacro:arg name="feedback_plot_csv_enabled" default="false" />
-    <xacro:arg name="feedback_plot_csv_file" default="/tmp/joint_monitor.csv" />
-    <xacro:arg name="feedback_plot_csv_append" default="false" />
+    <xacro:arg name="aux_joint_min" default="-0.69" />
+    <xacro:arg name="aux_joint_max" default="0.0" />
+    <xacro:arg name="arm_command_frame_format" default="legacy_position" />
+    <xacro:arg name="enable_dynamics_feedforward" default="false" />
+    <xacro:arg name="dynamics_mode" default="gravity" />
+    <xacro:arg name="dynamics_urdf_path" default="" />
+    <xacro:arg name="dynamics_feedforward_source" default="topic" />
+    <xacro:arg name="dynamics_feedforward_topic" default="/arm_dynamics/torques_nm" />
+    <xacro:arg name="dynamics_topic_timeout_sec" default="0.25" />
+    <xacro:arg name="dynamics_use_commanded_position" default="false" />
+    <xacro:arg name="dynamics_torque_scale" default="1.0" />
+    <xacro:arg name="dynamics_torque_limits_nm" default="0.5,0.5,0.3,0.2,0.15,0.1" />
+    <xacro:arg name="dynamics_torque_joint_signs" default="" />
+    <xacro:arg name="dynamics_torque_low_pass_alpha" default="0.2" />
     <!-- Import arm urdf file -->
     <xacro:include filename="$(find arm)/urdf/arm.urdf" />
@@ -72,11 +76,15 @@
       aux_joint_min="$(arg aux_joint_min)"
       aux_joint_max="$(arg aux_joint_max)"
-      enable_feedback_plot="$(arg enable_feedback_plot)"
-      feedback_plot_rate_hz="$(arg feedback_plot_rate_hz)"
-      feedback_plot_min_rad="$(arg feedback_plot_min_rad)"
-      feedback_plot_max_rad="$(arg feedback_plot_max_rad)"
-      feedback_plot_joint_filter="$(arg feedback_plot_joint_filter)"
-      feedback_plot_csv_enabled="$(arg feedback_plot_csv_enabled)"
-      feedback_plot_csv_file="$(arg feedback_plot_csv_file)"
-      feedback_plot_csv_append="$(arg feedback_plot_csv_append)"/>
+      arm_command_frame_format="$(arg arm_command_frame_format)"
+      enable_dynamics_feedforward="$(arg enable_dynamics_feedforward)"
+      dynamics_mode="$(arg dynamics_mode)"
+      dynamics_urdf_path="$(arg dynamics_urdf_path)"
+      dynamics_feedforward_source="$(arg dynamics_feedforward_source)"
+      dynamics_feedforward_topic="$(arg dynamics_feedforward_topic)"
+      dynamics_topic_timeout_sec="$(arg dynamics_topic_timeout_sec)"
+      dynamics_use_commanded_position="$(arg dynamics_use_commanded_position)"
+      dynamics_torque_scale="$(arg dynamics_torque_scale)"
+      dynamics_torque_limits_nm="$(arg dynamics_torque_limits_nm)"
+      dynamics_torque_joint_signs="$(arg dynamics_torque_joint_signs)"
+      dynamics_torque_low_pass_alpha="$(arg dynamics_torque_low_pass_alpha)"/>
 </robot>

Commit message: new urdf in

File: src/arm/urdf/arm.urdf (robot description, URDF)
Before this commit: robot arm, 10 links, 9 joints
Links:
- added link tool_base, mass 0.0983878201165868; collision mesh filename=package://arm/meshes/grippers/my_gripper_1/tool_base.STL; visual mesh filename=package://arm/meshes/grippers/my_gripper_1/tool_base.STL
- link base_link: mass 0.32006 -> 0.135833610555003; geometry collision mesh filename=package://arm/meshes/arm/base_link.STL; visual mesh filename=package://arm/meshes/arm/base_link.STL
- link link_1: mass 0.82985 -> 0.913798575246718; geometry collision mesh filename=package://arm/meshes/arm/link_1.STL; visual mesh filename=package://arm/meshes/arm/link_1.STL
- link link_2: mass 0.78271 -> 0.380008611681788; geometry collision mesh filename=package://arm/meshes/arm/link_2.STL; visual mesh filename=package://arm/meshes/arm/link_2.STL
- link link_3: mass 0.12605 -> 0.238605745340086; geometry collision mesh filename=package://arm/meshes/arm/link_3.STL; visual mesh filename=package://arm/meshes/arm/link_3.STL
- link link_4: mass 0.067165 -> 0.0708022799545759; geometry collision mesh filename=package://arm/meshes/arm/link_4.STL; visual mesh filename=package://arm/meshes/arm/link_4.STL
- link link_5: mass 0.060361 -> 0.0651571805551386; geometry collision mesh filename=package://arm/meshes/arm/link_5.STL; visual mesh filename=package://arm/meshes/arm/link_5.STL
- link link_6: mass 0.12546 -> 0.0245056804431765; geometry collision mesh filename=package://arm/meshes/arm/link_6.STL; visual mesh filename=package://arm/meshes/arm/link_6.STL
- link tool_link: mass 0.054319 -> 0.054318578390507; geometry collision mesh filename=package://arm/meshes/grippers/my_gripper_1/tool_link.STL; visual mesh filename=package://arm/meshes/grippers/my_gripper_1/tool_link.STL
Joints:
- added joint tool_base_fixed: type fixed, parent link_6, child tool_base, origin xyz=0 0 0 rpy=0 0 0
- joint joint_1: axis 0 0 -1 -> 0 0 1; limit lower=-3.14 upper=3.14 effort=0 velocity=2.0 -> lower=-3.1416 upper=3.1416 effort=0 velocity=0; origin xyz=0 0 0.105 rpy=0 0 0 -> xyz=0 0 -0.105 rpy=3.1416 0 0
- joint joint_2: limit lower=0.0 upper=3.14 effort=0 velocity=2.0 -> lower=0 upper=3.1416 effort=0 velocity=0; origin xyz=0.092 0 0 rpy=1.5708 0 1.5708 -> xyz=0 0 0 rpy=1.5708 0 -3.1416
- joint joint_3: limit lower=0.0 upper=3.14 effort=0 velocity=2.0 -> lower=-3.1416 upper=0 effort=0 velocity=0; origin xyz=0.65 0 -0.036 rpy=-3.1416 0 1.5708 -> xyz=0.65 0 0.056 rpy=0 0 1.5708
- joint joint_4: axis 0 0 1 -> 0 0 -1; limit lower=-3.14 upper=3.14 effort=0 velocity=2.0 -> lower=-3.1416 upper=3.1416 effort=0 velocity=0; origin xyz=0.045 -0.566 0 rpy=-1.5708 0 3.1416 -> xyz=0.045 0.566 0 rpy=1.5708 1.5708 0
- joint joint_5: limit lower=-3.14 upper=0.0 effort=0 velocity=2.0 -> lower=0 upper=3.1416 effort=0 velocity=0; origin xyz=0 0 0 rpy=1.5708 0 -1.5708 -> xyz=0 0 0 rpy=1.5708 -1.5708 0
- joint joint_6: limit lower=-3.14 upper=3.14 effort=0 velocity=2.0 -> lower=-3.1416 upper=3.1416 effort=0 velocity=0; origin xyz=0 0 0 rpy=1.5708 0 1.5708 -> xyz=0 -0.0475 0 rpy=1.5708 0 0
- joint tool_joint: limit lower=-0.69 upper=0.0 effort=0 velocity=2.0 -> lower=-0.69 upper=0.0 effort=0 velocity=0; origin xyz=-0.02305 0.00055 0.138 rpy=-1.5708 0 -3.1416 -> xyz=-0.02305 0.0029234 0.0895 rpy=1.5708 0 0; parent link_6 -> tool_base

File: src/arm_moveit_config/config/arm.ros2_control.xacro (robot description, xacro)
@@ -104,7 +104,7 @@
             <xacro:position_joint_interfaces joint_name="joint_1" initial_value="${initial_positions['joint_1']}" min_limit="-3.14" max_limit="3.14"/>
             <xacro:position_joint_interfaces joint_name="joint_2" initial_value="${initial_positions['joint_2']}" min_limit="0.0" max_limit="3.14"/>
-            <xacro:position_joint_interfaces joint_name="joint_3" initial_value="${initial_positions['joint_3']}" min_limit="0.0" max_limit="3.14"/>
+            <xacro:position_joint_interfaces joint_name="joint_3" initial_value="${initial_positions['joint_3']}" min_limit="-3.14" max_limit="0.0"/>
             <xacro:position_joint_interfaces joint_name="joint_4" initial_value="${initial_positions['joint_4']}" min_limit="-3.14" max_limit="3.14"/>
-            <xacro:position_joint_interfaces joint_name="joint_5" initial_value="${initial_positions['joint_5']}" min_limit="-3.14" max_limit="0.0"/>
+            <xacro:position_joint_interfaces joint_name="joint_5" initial_value="${initial_positions['joint_5']}" min_limit="0.0" max_limit="3.14"/>
             <xacro:position_joint_interfaces joint_name="joint_6" initial_value="${initial_positions['joint_6']}" min_limit="-3.14" max_limit="3.14"/>
             <xacro:position_joint_interfaces joint_name="tool_joint" initial_value="${initial_positions['tool_joint']}" min_limit="${aux_joint_min}" max_limit="${aux_joint_max}"/>

File: src/arm_moveit_config/config/arm.urdf.xacro (robot description, xacro)
@@ -28,6 +28,6 @@
     <xacro:arg name="dynamics_torque_joint_signs" default="" />
     <xacro:arg name="dynamics_torque_low_pass_alpha" default="0.2" />
-    <!-- Import arm urdf file -->
-    <xacro:include filename="$(find arm)/urdf/arm.urdf" />
+    <!-- Import the modular arm + selected gripper model. -->
+    <xacro:include filename="$(find arm)/urdf/arm.urdf.xacro" />
     <!-- Import control_xacro -->
     <xacro:include filename="arm.ros2_control.xacro" />
@@ -38,6 +38,6 @@
       name="limit_z_max"
       parent_link="uav_mount"
-      xyz="0 0 0.05"
-      rpy="0 0 1.57"
+      xyz="0 0 0.005"
+      rpy="0 0 0"
       size="0.4 0.64 0.01"
       color="0.9 0.1 0.1 0.2"
@@ -46,6 +46,6 @@
       name="limit_y_min"
       parent_link="uav_mount"
-      xyz="0.32 0 -0.75"
-      rpy="1.57 0 1.57"
+      xyz="0 -0.32 -0.75"
+      rpy="1.57 0 0"
       size="0.4 1.6 0.01"
       color="0.9 0.1 0.1 0.2"
@@ -54,6 +54,6 @@
       name="limit_y_max"
       parent_link="uav_mount"
-      xyz="-0.32 0 -0.75"
-      rpy="1.57 0 1.57"
+      xyz="0 0.32 -0.75"
+      rpy="1.57 0 0"
       size="0.4 1.6 0.01"
       color="0.9 0.1 0.1 0.2"

Commit message: 1

File: src/arm/urdf/arm.urdf (robot description, URDF)
Before this commit: robot arm, 11 links, 10 joints
Joints:
- joint joint_1: limit lower=-3.1416 upper=3.1416 effort=0 velocity=0 -> lower=-3.1416 upper=3.1416 effort=100 velocity=2.0
- joint joint_2: limit lower=0 upper=3.1416 effort=0 velocity=0 -> lower=0 upper=3.1416 effort=100 velocity=2.0
- joint joint_3: limit lower=-3.1416 upper=0 effort=0 velocity=0 -> lower=-3.1416 upper=0 effort=100 velocity=2.0
- joint joint_4: limit lower=-3.1416 upper=3.1416 effort=0 velocity=0 -> lower=-3.1416 upper=3.1416 effort=100 velocity=2.0
- joint joint_5: limit lower=0 upper=3.1416 effort=0 velocity=0 -> lower=0 upper=3.1416 effort=100 velocity=2.0
- joint joint_6: limit lower=-3.1416 upper=3.1416 effort=0 velocity=0 -> lower=-3.1416 upper=3.1416 effort=100 velocity=2.0
- joint tool_joint: limit lower=-0.69 upper=0.0 effort=0 velocity=0 -> lower=-0.69 upper=0.0 effort=20 velocity=2.0

File: src/arm/urdf/arm_core.urdf.xacro (robot description, xacro)
@@ -100,6 +100,6 @@
       lower="-3.1416"
       upper="3.1416"
-      effort="0"
-      velocity="0" />
+      effort="100"
+      velocity="2.0" />
   </joint>
   <link
@@ -158,6 +158,6 @@
       lower="0"
       upper="3.1416"
-      effort="0"
-      velocity="0" />
+      effort="100"
+      velocity="2.0" />
   </joint>
   <link
@@ -216,6 +216,6 @@
       lower="-3.1416"
       upper="0"
-      effort="0"
-      velocity="0" />
+      effort="100"
+      velocity="2.0" />
   </joint>
   <link
@@ -274,6 +274,6 @@
       lower="-3.1416"
       upper="3.1416"
-      effort="0"
-      velocity="0" />
+      effort="100"
+      velocity="2.0" />
   </joint>
   <link
@@ -332,6 +332,6 @@
       lower="0"
       upper="3.1416"
-      effort="0"
-      velocity="0" />
+      effort="100"
+      velocity="2.0" />
   </joint>
   <link
@@ -390,6 +390,6 @@
       lower="-3.1416"
       upper="3.1416"
-      effort="0"
-      velocity="0" />
+      effort="100"
+      velocity="2.0" />
   </joint>
   </xacro:macro>

File: src/arm/urdf/grippers/my_gripper_1.urdf.xacro (robot description, xacro)
@@ -105,6 +105,6 @@
       lower="${tool_joint_min}"
       upper="${tool_joint_max}"
-      effort="0"
-      velocity="0" />
+      effort="20"
+      velocity="2.0" />
   </joint>
   </xacro:macro>

File: src/arm_moveit_config/config/arm.ros2_control.xacro (robot description, xacro)
@@ -2,5 +2,5 @@
 <robot xmlns:xacro="http://www.ros.org/wiki/xacro">
     <xacro:arg name="use_fake_hardware" default="true"/>
-    <xacro:arg name="serial_port" default="/dev/ttyUSB4"/>
+    <xacro:arg name="serial_port" default="/dev/ttyACM0"/>
     <xacro:arg name="reader_port" default="/dev/ttyUSB5"/>
     <xacro:arg name="gripper_port" default="/dev/ttyUSB6"/>
@@ -16,4 +16,11 @@
     <xacro:arg name="aux_joint_max" default="0.0"/>
     <xacro:arg name="arm_command_frame_format" default="legacy_position"/>
+    <xacro:arg name="stm32_control_mode" default="0"/>
+    <xacro:arg name="stm32_kp" default="50,50,50,50,50,50"/>
+    <xacro:arg name="stm32_kd" default="2,2,2,2,2,2"/>
+    <xacro:arg name="stm32_heartbeat_duration_sec" default="1.0"/>
+    <xacro:arg name="stm32_trigger_duration_sec" default="3.0"/>
+    <xacro:arg name="stm32_feedback_wait_timeout_sec" default="2.0"/>
+    <xacro:arg name="enable_stm32_zero_trigger" default="false"/>
     <xacro:arg name="enable_dynamics_feedforward" default="false"/>
     <xacro:arg name="dynamics_mode" default="gravity"/>
@@ -36,4 +43,5 @@
             </state_interface>
             <state_interface name="velocity"/>
+            <state_interface name="effort"/>
         </joint>
     </xacro:macro>
@@ -42,5 +50,5 @@
         initial_positions_file
         use_fake_hardware:=true
-        serial_port:='/dev/ttyUSB4'
+        serial_port:='/dev/ttyACM0'
         reader_port:='/dev/ttyUSB5'
         gripper_port:='/dev/ttyUSB6'
@@ -56,4 +64,11 @@
         aux_joint_max:='0.0'
         arm_command_frame_format:='legacy_position'
+        stm32_control_mode:='0'
+        stm32_kp:='50,50,50,50,50,50'
+        stm32_kd:='2,2,2,2,2,2'
+        stm32_heartbeat_duration_sec:='1.0'
+        stm32_trigger_duration_sec:='3.0'
+        stm32_feedback_wait_timeout_sec:='2.0'
+        enable_stm32_zero_trigger:='false'
         enable_dynamics_feedforward:='false'
         dynamics_mode:='gravity'
@@ -89,4 +104,11 @@
                     <param name="aux_joint_max">${aux_joint_max}</param>
                     <param name="arm_command_frame_format">${arm_command_frame_format}</param>
+                    <param name="stm32_control_mode">${stm32_control_mode}</param>
+                    <param name="stm32_kp">${stm32_kp}</param>
+                    <param name="stm32_kd">${stm32_kd}</param>
+                    <param name="stm32_heartbeat_duration_sec">${stm32_heartbeat_duration_sec}</param>
+                    <param name="stm32_trigger_duration_sec">${stm32_trigger_duration_sec}</param>
+                    <param name="stm32_feedback_wait_timeout_sec">${stm32_feedback_wait_timeout_sec}</param>
+                    <param name="enable_stm32_zero_trigger">${enable_stm32_zero_trigger}</param>
                     <param name="enable_dynamics_feedforward">${enable_dynamics_feedforward}</param>
                     <param name="dynamics_mode">${dynamics_mode}</param>

File: src/arm_moveit_config/config/arm.urdf.xacro (robot description, xacro)
@@ -3,5 +3,5 @@
     <xacro:arg name="initial_positions_file" default="initial_positions.yaml" />
     <xacro:arg name="use_fake_hardware" default="true" />
-    <xacro:arg name="serial_port" default="/dev/ttyUSB4" />
+    <xacro:arg name="serial_port" default="/dev/ttyACM0" />
     <xacro:arg name="reader_port" default="/dev/ttyUSB5" />
     <xacro:arg name="gripper_port" default="/dev/ttyUSB6" />
@@ -17,4 +17,11 @@
     <xacro:arg name="aux_joint_max" default="0.0" />
     <xacro:arg name="arm_command_frame_format" default="legacy_position" />
+    <xacro:arg name="stm32_control_mode" default="0" />
+    <xacro:arg name="stm32_kp" default="50,50,50,50,50,50" />
+    <xacro:arg name="stm32_kd" default="2,2,2,2,2,2" />
+    <xacro:arg name="stm32_heartbeat_duration_sec" default="1.0" />
+    <xacro:arg name="stm32_trigger_duration_sec" default="3.0" />
+    <xacro:arg name="stm32_feedback_wait_timeout_sec" default="2.0" />
+    <xacro:arg name="enable_stm32_zero_trigger" default="false" />
     <xacro:arg name="enable_dynamics_feedforward" default="false" />
     <xacro:arg name="dynamics_mode" default="gravity" />
@@ -77,4 +84,11 @@
       aux_joint_max="$(arg aux_joint_max)"
       arm_command_frame_format="$(arg arm_command_frame_format)"
+      stm32_control_mode="$(arg stm32_control_mode)"
+      stm32_kp="$(arg stm32_kp)"
+      stm32_kd="$(arg stm32_kd)"
+      stm32_heartbeat_duration_sec="$(arg stm32_heartbeat_duration_sec)"
+      stm32_trigger_duration_sec="$(arg stm32_trigger_duration_sec)"
+      stm32_feedback_wait_timeout_sec="$(arg stm32_feedback_wait_timeout_sec)"
+      enable_stm32_zero_trigger="$(arg enable_stm32_zero_trigger)"
       enable_dynamics_feedforward="$(arg enable_dynamics_feedforward)"
       dynamics_mode="$(arg dynamics_mode)"
