Commit message: 1

File: src/arm/urdf/arm.urdf (robot description, URDF)
Before this commit: robot arm, 11 links, 10 joints
Joints:
- joint tool0_fixed: origin xyz=0 0.01 0.2 rpy=0 0 0 -> xyz=-0.03 0 0.018 rpy=0 0 0

File: src/arm/urdf/arm.urdf.xacro (robot description, xacro)
@@ -17,5 +17,5 @@
     <parent link="link_6"/>
     <child link="tool0"/>
-    <origin xyz="0 0.01 0.2" rpy="0 0 0"/>
+    <origin rpy="0 0 0" xyz="-0.03 0 0.18"/>
   </joint>
   <xacro:my_gripper_1

File: src/arm/urdf/arm_core.urdf.xacro (robot description, xacro)
@@ -333,5 +333,5 @@
       upper="3.1416"
       effort="100"
-      velocity="2.0" />
+      velocity="1.0" />
   </joint>
   <link

File: src/arm_moveit_config/config/arm.ros2_control.xacro (robot description, xacro)
@@ -19,8 +19,11 @@
     <xacro:arg name="stm32_kp" default="50,50,50,50,50,50"/>
     <xacro:arg name="stm32_kd" default="2,2,2,2,2,2"/>
+    <xacro:arg name="stm32_v_des_limits_rad_s" default="1,1,1,1,1,1"/>
     <xacro:arg name="stm32_heartbeat_duration_sec" default="1.0"/>
     <xacro:arg name="stm32_trigger_duration_sec" default="3.0"/>
     <xacro:arg name="stm32_feedback_wait_timeout_sec" default="2.0"/>
     <xacro:arg name="enable_stm32_zero_trigger" default="false"/>
+    <xacro:arg name="stm32_recover_safe_drop_on_start" default="true"/>
+    <xacro:arg name="stm32_recover_duration_sec" default="0.25"/>
     <xacro:arg name="stm32_trace_enabled" default="false"/>
     <xacro:arg name="stm32_trace_directory" default="/tmp/arm_stm32_traces"/>
@@ -43,4 +46,5 @@
         <joint name="${joint_name}">
             <command_interface name="position"/>
+            <command_interface name="velocity"/>
             <param name="min">${min_limit}</param>
             <param name="max">${max_limit}</param>
@@ -73,8 +77,11 @@
         stm32_kp:='50,50,50,50,50,50'
         stm32_kd:='2,2,2,2,2,2'
+        stm32_v_des_limits_rad_s:='1,1,1,1,1,1'
         stm32_heartbeat_duration_sec:='1.0'
         stm32_trigger_duration_sec:='3.0'
         stm32_feedback_wait_timeout_sec:='2.0'
         enable_stm32_zero_trigger:='false'
+        stm32_recover_safe_drop_on_start:='true'
+        stm32_recover_duration_sec:='0.25'
         stm32_trace_enabled:='false'
         stm32_trace_directory:='/tmp/arm_stm32_traces'
@@ -119,8 +126,11 @@
                     <param name="stm32_kp">${stm32_kp}</param>
                     <param name="stm32_kd">${stm32_kd}</param>
+                    <param name="stm32_v_des_limits_rad_s">${stm32_v_des_limits_rad_s}</param>
                     <param name="stm32_heartbeat_duration_sec">${stm32_heartbeat_duration_sec}</param>
                     <param name="stm32_trigger_duration_sec">${stm32_trigger_duration_sec}</param>
                     <param name="stm32_feedback_wait_timeout_sec">${stm32_feedback_wait_timeout_sec}</param>
                     <param name="enable_stm32_zero_trigger">${enable_stm32_zero_trigger}</param>
+                    <param name="stm32_recover_safe_drop_on_start">${stm32_recover_safe_drop_on_start}</param>
+                    <param name="stm32_recover_duration_sec">${stm32_recover_duration_sec}</param>
                     <param name="stm32_trace_enabled">${stm32_trace_enabled}</param>
                     <param name="stm32_trace_directory">${stm32_trace_directory}</param>

File: src/arm_moveit_config/config/arm.urdf.xacro (robot description, xacro)
@@ -20,8 +20,11 @@
     <xacro:arg name="stm32_kp" default="50,50,50,50,50,50" />
     <xacro:arg name="stm32_kd" default="2,2,2,2,2,2" />
+    <xacro:arg name="stm32_v_des_limits_rad_s" default="1,1,1,1,1,1" />
     <xacro:arg name="stm32_heartbeat_duration_sec" default="1.0" />
     <xacro:arg name="stm32_trigger_duration_sec" default="3.0" />
     <xacro:arg name="stm32_feedback_wait_timeout_sec" default="2.0" />
     <xacro:arg name="enable_stm32_zero_trigger" default="false" />
+    <xacro:arg name="stm32_recover_safe_drop_on_start" default="true" />
+    <xacro:arg name="stm32_recover_duration_sec" default="0.25" />
     <xacro:arg name="stm32_trace_enabled" default="false" />
     <xacro:arg name="stm32_trace_directory" default="/tmp/arm_stm32_traces" />
@@ -93,8 +96,11 @@
       stm32_kp="$(arg stm32_kp)"
       stm32_kd="$(arg stm32_kd)"
+      stm32_v_des_limits_rad_s="$(arg stm32_v_des_limits_rad_s)"
       stm32_heartbeat_duration_sec="$(arg stm32_heartbeat_duration_sec)"
       stm32_trigger_duration_sec="$(arg stm32_trigger_duration_sec)"
       stm32_feedback_wait_timeout_sec="$(arg stm32_feedback_wait_timeout_sec)"
       enable_stm32_zero_trigger="$(arg enable_stm32_zero_trigger)"
+      stm32_recover_safe_drop_on_start="$(arg stm32_recover_safe_drop_on_start)"
+      stm32_recover_duration_sec="$(arg stm32_recover_duration_sec)"
       stm32_trace_enabled="$(arg stm32_trace_enabled)"
       stm32_trace_directory="$(arg stm32_trace_directory)"

Commit message: fix speed imits

File: src/arm/urdf/arm.urdf (robot description, URDF)
Before this commit: robot arm, 11 links, 10 joints
Joints:
- joint joint_3: limit lower=-3.1416 upper=0 effort=100 velocity=2.0 -> lower=-3.1416 upper=0 effort=100 velocity=0.5
- joint joint_5: limit lower=0 upper=3.1416 effort=100 velocity=2.0 -> lower=0 upper=3.1416 effort=100 velocity=1.0

File: src/arm/urdf/arm_core.urdf.xacro (robot description, xacro)
@@ -217,5 +217,5 @@
       upper="0"
       effort="100"
-      velocity="2.0" />
+      velocity="0.5" />
   </joint>
   <link

File: src/arm_moveit_config/config/arm.ros2_control.xacro (robot description, xacro)
@@ -24,4 +24,7 @@
     <xacro:arg name="hw_slowdown" default="10"/>
     <xacro:arg name="feedback_velocity_low_pass_alpha" default="1,1,1,1,1,1"/>
+    <xacro:arg name="enable_arm_command_limiter" default="true"/>
+    <xacro:arg name="arm_command_velocity_limits_rad_s" default="2.0,2.0,0.5,2.0,1.0,2.0"/>
+    <xacro:arg name="arm_command_acceleration_limits_rad_s2" default="1.0,1.0,0.2,1.0,0.5,1.0"/>
     <xacro:arg name="initial_read_timeout_sec" default="2.0"/>
     <xacro:arg name="first_power_on" default="true"/>
@@ -32,5 +35,5 @@
     <xacro:arg name="stm32_kp" default="50,50,50,50,50,50"/>
     <xacro:arg name="stm32_kd" default="2,2,2,2,2,2"/>
-    <xacro:arg name="stm32_v_des_limits_rad_s" default="1,1,1,1,1,1"/>
+    <xacro:arg name="stm32_v_des_limits_rad_s" default="2.0,2.0,0.5,2.0,1.0,2.0"/>
     <xacro:arg name="stm32_heartbeat_duration_sec" default="1.0"/>
     <xacro:arg name="stm32_trigger_duration_sec" default="3.0"/>
@@ -95,4 +98,7 @@
         hw_slowdown:='10'
         feedback_velocity_low_pass_alpha:='1,1,1,1,1,1'
+        enable_arm_command_limiter:='true'
+        arm_command_velocity_limits_rad_s:='2.0,2.0,0.5,2.0,1.0,2.0'
+        arm_command_acceleration_limits_rad_s2:='1.0,1.0,0.2,1.0,0.5,1.0'
         initial_read_timeout_sec:='2.0'
         first_power_on:='true'
@@ -103,5 +109,5 @@
         stm32_kp:='50,50,50,50,50,50'
         stm32_kd:='2,2,2,2,2,2'
-        stm32_v_des_limits_rad_s:='1,1,1,1,1,1'
+        stm32_v_des_limits_rad_s:='2.0,2.0,0.5,2.0,1.0,2.0'
         stm32_heartbeat_duration_sec:='1.0'
         stm32_trigger_duration_sec:='3.0'
@@ -157,4 +163,7 @@
                     <param name="hw_slowdown">${hw_slowdown}</param>
                     <param name="feedback_velocity_low_pass_alpha">${feedback_velocity_low_pass_alpha}</param>
+                    <param name="enable_arm_command_limiter">${enable_arm_command_limiter}</param>
+                    <param name="arm_command_velocity_limits_rad_s">${arm_command_velocity_limits_rad_s}</param>
+                    <param name="arm_command_acceleration_limits_rad_s2">${arm_command_acceleration_limits_rad_s2}</param>
                     <param name="initial_read_timeout_sec">${initial_read_timeout_sec}</param>
                     <param name="first_power_on">${first_power_on}</param>

File: src/arm_moveit_config/config/arm.urdf.xacro (robot description, xacro)
@@ -25,4 +25,7 @@
     <xacro:arg name="hw_slowdown" default="10" />
     <xacro:arg name="feedback_velocity_low_pass_alpha" default="1,1,1,1,1,1" />
+    <xacro:arg name="enable_arm_command_limiter" default="true" />
+    <xacro:arg name="arm_command_velocity_limits_rad_s" default="2.0,2.0,0.5,2.0,1.0,2.0" />
+    <xacro:arg name="arm_command_acceleration_limits_rad_s2" default="1.0,1.0,0.2,1.0,0.5,1.0" />
     <xacro:arg name="initial_read_timeout_sec" default="2.0" />
     <xacro:arg name="first_power_on" default="true" />
@@ -33,5 +36,5 @@
     <xacro:arg name="stm32_kp" default="50,50,50,50,50,50" />
     <xacro:arg name="stm32_kd" default="2,2,2,2,2,2" />
-    <xacro:arg name="stm32_v_des_limits_rad_s" default="1,1,1,1,1,1" />
+    <xacro:arg name="stm32_v_des_limits_rad_s" default="2.0,2.0,0.5,2.0,1.0,2.0" />
     <xacro:arg name="stm32_heartbeat_duration_sec" default="1.0" />
     <xacro:arg name="stm32_trigger_duration_sec" default="3.0" />
@@ -114,4 +117,7 @@
       hw_slowdown="$(arg hw_slowdown)"
       feedback_velocity_low_pass_alpha="$(arg feedback_velocity_low_pass_alpha)"
+      enable_arm_command_limiter="$(arg enable_arm_command_limiter)"
+      arm_command_velocity_limits_rad_s="$(arg arm_command_velocity_limits_rad_s)"
+      arm_command_acceleration_limits_rad_s2="$(arg arm_command_acceleration_limits_rad_s2)"
       initial_read_timeout_sec="$(arg initial_read_timeout_sec)"
       first_power_on="$(arg first_power_on)"

Commit message: match new speed

File: src/arm/urdf/arm.urdf (robot description, URDF)
Before this commit: robot arm, 11 links, 10 joints
Joints:
- joint joint_1: limit lower=-3.1416 upper=3.1416 effort=100 velocity=2.0 -> lower=-3.1416 upper=3.1416 effort=100 velocity=0.20
- joint joint_2: limit lower=0 upper=3.1416 effort=100 velocity=2.0 -> lower=0 upper=3.1416 effort=100 velocity=0.20
- joint joint_3: limit lower=-3.1416 upper=0 effort=100 velocity=0.5 -> lower=-3.1416 upper=0 effort=100 velocity=0.10
- joint joint_4: limit lower=-3.1416 upper=3.1416 effort=100 velocity=2.0 -> lower=-3.1416 upper=3.1416 effort=100 velocity=0.20
- joint joint_5: limit lower=0 upper=3.1416 effort=100 velocity=1.0 -> lower=0 upper=3.1416 effort=100 velocity=0.10
- joint joint_6: limit lower=-3.1416 upper=3.1416 effort=100 velocity=2.0 -> lower=-3.1416 upper=3.1416 effort=100 velocity=0.20

File: src/arm/urdf/arm_core.urdf.xacro (robot description, xacro)
@@ -101,5 +101,5 @@
       upper="3.1416"
       effort="100"
-      velocity="2.0" />
+      velocity="0.20" />
   </joint>
   <link
@@ -159,5 +159,5 @@
       upper="3.1416"
       effort="100"
-      velocity="2.0" />
+      velocity="0.20" />
   </joint>
   <link
@@ -217,5 +217,5 @@
       upper="0"
       effort="100"
-      velocity="0.5" />
+      velocity="0.10" />
   </joint>
   <link
@@ -275,5 +275,5 @@
       upper="3.1416"
       effort="100"
-      velocity="2.0" />
+      velocity="0.20" />
   </joint>
   <link
@@ -333,5 +333,5 @@
       upper="3.1416"
       effort="100"
-      velocity="1.0" />
+      velocity="0.10" />
   </joint>
   <link
@@ -391,5 +391,5 @@
       upper="3.1416"
       effort="100"
-      velocity="2.0" />
+      velocity="0.20" />
   </joint>
   </xacro:macro>

File: src/arm_moveit_config/config/arm.ros2_control.xacro (robot description, xacro)
@@ -25,6 +25,6 @@
     <xacro:arg name="feedback_velocity_low_pass_alpha" default="1,1,1,1,1,1"/>
     <xacro:arg name="enable_arm_command_limiter" default="true"/>
-    <xacro:arg name="arm_command_velocity_limits_rad_s" default="2.0,2.0,0.5,2.0,1.0,2.0"/>
-    <xacro:arg name="arm_command_acceleration_limits_rad_s2" default="1.0,1.0,0.2,1.0,0.5,1.0"/>
+    <xacro:arg name="arm_command_velocity_limits_rad_s" default="0.20,0.20,0.10,0.20,0.10,0.20"/>
+    <xacro:arg name="arm_command_acceleration_limits_rad_s2" default="0.10,0.10,0.10,0.10,0.10,0.10"/>
     <xacro:arg name="initial_read_timeout_sec" default="2.0"/>
     <xacro:arg name="first_power_on" default="true"/>
@@ -35,5 +35,5 @@
     <xacro:arg name="stm32_kp" default="50,50,50,50,50,50"/>
     <xacro:arg name="stm32_kd" default="2,2,2,2,2,2"/>
-    <xacro:arg name="stm32_v_des_limits_rad_s" default="2.0,2.0,0.5,2.0,1.0,2.0"/>
+    <xacro:arg name="stm32_v_des_limits_rad_s" default="0.20,0.20,0.10,0.20,0.10,0.20"/>
     <xacro:arg name="stm32_heartbeat_duration_sec" default="1.0"/>
     <xacro:arg name="stm32_trigger_duration_sec" default="3.0"/>
@@ -99,6 +99,6 @@
         feedback_velocity_low_pass_alpha:='1,1,1,1,1,1'
         enable_arm_command_limiter:='true'
-        arm_command_velocity_limits_rad_s:='2.0,2.0,0.5,2.0,1.0,2.0'
-        arm_command_acceleration_limits_rad_s2:='1.0,1.0,0.2,1.0,0.5,1.0'
+        arm_command_velocity_limits_rad_s:='0.20,0.20,0.10,0.20,0.10,0.20'
+        arm_command_acceleration_limits_rad_s2:='0.10,0.10,0.10,0.10,0.10,0.10'
         initial_read_timeout_sec:='2.0'
         first_power_on:='true'
@@ -109,5 +109,5 @@
         stm32_kp:='50,50,50,50,50,50'
         stm32_kd:='2,2,2,2,2,2'
-        stm32_v_des_limits_rad_s:='2.0,2.0,0.5,2.0,1.0,2.0'
+        stm32_v_des_limits_rad_s:='0.20,0.20,0.10,0.20,0.10,0.20'
         stm32_heartbeat_duration_sec:='1.0'
         stm32_trigger_duration_sec:='3.0'

File: src/arm_moveit_config/config/arm.urdf.xacro (robot description, xacro)
@@ -26,6 +26,6 @@
     <xacro:arg name="feedback_velocity_low_pass_alpha" default="1,1,1,1,1,1" />
     <xacro:arg name="enable_arm_command_limiter" default="true" />
-    <xacro:arg name="arm_command_velocity_limits_rad_s" default="2.0,2.0,0.5,2.0,1.0,2.0" />
-    <xacro:arg name="arm_command_acceleration_limits_rad_s2" default="1.0,1.0,0.2,1.0,0.5,1.0" />
+    <xacro:arg name="arm_command_velocity_limits_rad_s" default="0.20,0.20,0.10,0.20,0.10,0.20" />
+    <xacro:arg name="arm_command_acceleration_limits_rad_s2" default="0.10,0.10,0.10,0.10,0.10,0.10" />
     <xacro:arg name="initial_read_timeout_sec" default="2.0" />
     <xacro:arg name="first_power_on" default="true" />
@@ -36,5 +36,5 @@
     <xacro:arg name="stm32_kp" default="50,50,50,50,50,50" />
     <xacro:arg name="stm32_kd" default="2,2,2,2,2,2" />
-    <xacro:arg name="stm32_v_des_limits_rad_s" default="2.0,2.0,0.5,2.0,1.0,2.0" />
+    <xacro:arg name="stm32_v_des_limits_rad_s" default="0.20,0.20,0.10,0.20,0.10,0.20" />
     <xacro:arg name="stm32_heartbeat_duration_sec" default="1.0" />
     <xacro:arg name="stm32_trigger_duration_sec" default="3.0" />
